File: KiCad/ZeDMD_WiFi/ZeDMD.kicad_sch (KiCad schematic)
At the start: 5 parts, among them J9 Conn_02x08_Odd_Even, SW1 Menu Left, SW2 Boot/Value+, SW3 Value-, SW4 Menu Right

Commit message: Update PCB to Rev1.3
Changed lines of the file:
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@@
 	(title_block
 		(title "HUB75")
-		(date "2026-07-11")
-		(rev "1.2")
+		(date "2026-09-04")
+		(rev "1.3")
 		(company "elabree")
-		(comment 1 "https://github.com/jens-b/ZeDMD-5.1.8-WIFI-128x32")
+		(comment 1 "https://github.com/jens-b/The-Arcade")
 		(comment 2 "https://ppuc.github.io/docs/zedmd/")
 		(comment 3 "https://github.com/PPUC/ZeDMD")
@@
 	(wire
 		(pts
+			(xy 0.0762 0.0762) (xy 78.8162 0.0762)
+		)
+		(stroke
+			(width 0)
+			(type default)
+		)
+	)
+	(wire
+		(pts
 			(xy 138.43 85.09) (xy 157.48 85.09)
 		)
@@
 		)
 		(stroke
+			(width 0)
+			(type default)
+		)
+	)
+	(wire
+		(pts
+			(xy 78.8162 0.0762) (xy 78.8162 20.3962)
+		)
+		(stroke
