File: KiCad/ZeDMD_WiFi/ZeDMD_WiFi.kicad_pcb (KiCad board)
At the start: 2 copper layers, 1 part, among them U1 ESP32-S3-DevKitC

Commit message: Initial setup
Parts:
- removed U1: ESP32-S3-DevKitC, PCM_Espressif:ESP32-S3-DevKitC
Other:
- board outline added: 100 x 80 mm
- board text added: "+5V"
- board text added: "1"
- board text added: "CLK"
- board text added: "CS"
- board text added: "GND"
- board text added: "HUB75-E"
- board text added: "INT"
- board text added: "MISO"
- board text added: "MOSI"
- board text added: "Rev: 1.0"
- board text added: "ZeDMD_ESP32-S3"
- board text added: "https://ppuc.github.io/docs/"

Commit message: Placement V1.1
Parts:
- added D1: 1N5819, Diode_THT:D_DO-41_SOD81_P10.16mm_Horizontal, F.Cu at (172.1, 82.5)
- added D2: 1N5822, Diode_THT:D_DO-201AD_P15.24mm_Horizontal, F.Cu at (234.5, 136.1)
- added J1: max98357-L, Connector_PinSocket_2.54mm:PinSocket_1x07_P2.54mm_Vertical, F.Cu at (163.0, 102.0)
- added J10: Conn_01x02_Pin, Connector_PinHeader_2.54mm:PinHeader_1x02_P2.54mm_Vertical, F.Cu at (167.7, 106.0)
- added J11: Conn_01x02_Pin, Connector_PinHeader_2.54mm:PinHeader_1x02_P2.54mm_Vertical, F.Cu at (188.2, 106.0)
- added J2: MicroSD, Connector_PinSocket_2.54mm:PinSocket_1x06_P2.54mm_Vertical, F.Cu at (204.5, 87.4)
- added J3: max98357-R, Connector_PinSocket_2.54mm:PinSocket_1x07_P2.54mm_Vertical, F.Cu at (182.9, 102.0)
- added J4: MAX_Vin_SELECT, Connector_PinHeader_2.54mm:PinHeader_2x03_P2.54mm_Vertical, F.Cu at (156.9, 78.8)
- added J5: RGBout_SELECT, Connector_PinHeader_2.54mm:PinHeader_1x03_P2.54mm_Vertical, F.Cu at (219.5, 108.5)
- added J6: 5Vin_OPTION, Connector_PinHeader_2.54mm:PinHeader_1x02_P2.54mm_Vertical, F.Cu at (220.8, 132.8)
- added J7: 5V, ZeDMD_WiFi:KF7.62_2P, F.Cu at (217.0, 142.0)
- added J8: USB-C breakout, Connector_PinSocket_2.54mm:PinSocket_1x06_P2.54mm_Vertical, F.Cu at (157.2, 102.5)
- added J9: Conn_02x08_Odd_Even, Connector_IDC:IDC-Header_2x08_P2.54mm_Vertical, F.Cu at (160.9, 143.5)
- added R1: 100k, Resistor_THT:R_Axial_DIN0207_L6.3mm_D2.5mm_P10.16mm_Horizontal, F.Cu at (175.9, 82.5)
- added R2: 680k, Resistor_THT:R_Axial_DIN0207_L6.3mm_D2.5mm_P10.16mm_Horizontal, F.Cu at (188.9, 82.5)
- added R3: 10k, Resistor_THT:R_Axial_DIN0207_L6.3mm_D2.5mm_P10.16mm_Horizontal, F.Cu at (154.4, 72.0)
- added SW1: Menu Left, Button_Switch_THT:SW_PUSH_6mm, F.Cu at (215.0, 73.0)
- added SW2: Boot/Value+, Button_Switch_THT:SW_PUSH_6mm, F.Cu at (200.0, 73.0)
- added SW3: Value-, Button_Switch_THT:SW_PUSH_6mm, F.Cu at (185.0, 73.0)
- added SW4: Menu Right, Button_Switch_THT:SW_PUSH_6mm, F.Cu at (170.0, 73.0)
- added TP1: TestPoint, Connector_PinHeader_2.54mm:PinHeader_1x01_P2.54mm_Vertical, F.Cu at (190.0, 142.0)
- added U1: ESP32-S3-DevKitC, PCM_Espressif:ESP32-S3-DevKitC, F.Cu at (150.6, 132.4)
Routing:
- added copper zone on In1.Cu, net GND
Other:
- outline, holes or cut-outs redrawn
- copper layers 2 -> 4
- board text added: "Rev: 1.1"
- board text added: "ZeDMD_WiFi; ESP32-S3"
- board text removed: "CLK"
- board text removed: "CS"
- board text removed: "INT"
- board text removed: "MISO"
- board text removed: "MOSI"
- board text removed: "Rev: 1.0"
- board text removed: "ZeDMD_ESP32-S3"

Commit message: Placement ready
Parts:
- added TP2: Vin, Connector_PinHeader_2.54mm:PinHeader_1x01_P2.54mm_Vertical, F.Cu at (178.2, 106.0)
- added TP3: Vin, Connector_PinHeader_2.54mm:PinHeader_1x01_P2.54mm_Vertical, F.Cu at (198.2, 106.0)
- added TP4: GND, Connector_PinHeader_2.54mm:PinHeader_1x01_P2.54mm_Vertical, F.Cu at (150.0, 82.5)
- J7: value 5V -> KF7.62 Barrier Terminal Block 2P
- R2: value 680k -> 390k
- TP1: value TestPoint -> GND
- moved J11 2.75 mm to (185.5, 106.0)
- moved J10 2.00 mm to (165.7, 106.0)
- moved TP1 1.41 mm to (189.0, 141.0)
Connections:
- net Net-(D2-A) renamed /RGBout
- J10 pad 1: unconnected-(J10-Pin_1-Pad1) -> GND
- J11 pad 1: unconnected-(J11-Pin_1-Pad1) -> GND
Routing:
- net /ESP32-S3-DevKitC-1-N16R8/ESP5V: track 0.00 -> 153.6 mm, vias 0 -> 3
- net /VBUS: track 0.00 -> 117.6 mm
- net /MAX_Vin: track 0.00 -> 101.6 mm, vias 0 -> 1
- net +3.3V: track 0.00 -> 69.7 mm
- net /RGBout: track 0.00 -> 22.6 mm
- net /SD_R: track 0.00 -> 21.2 mm
- net /SD_L: track 0.00 -> 20.7 mm
- net /RGBout_5Vin: track 0.00 -> 20.3 mm
- net GND: track 0.00 -> 11.6 mm
- net /GAIN_R: track 0.00 -> 5.03 mm
- net /GAIN_L: track 0.00 -> 4.96 mm
- added copper zone on In2.Cu, net GND
Other:
- board text added: "ENABLE 5V input"
- board text added: "ESP5V"
- board text added: "USB-C"
- board text added: "ZeDMD"
- board text added: "gain"
- board text added: "https://github.com/jens-b/ZeDMD-5.1.8-WIFI-128x32"
- board text removed: "https://ppuc.github.io/docs/"

Commit message: Routing
Parts:
- moved J11 2.49 mm to (188.0, 106.2)
- moved TP1 2.47 mm to (191.1, 142.2)
- moved J10 2.18 mm to (167.9, 106.2)
- moved J9 1.01 mm to (161.9, 143.5)
- moved U1 0.31 mm to (150.5, 132.7)
- moved TP2 0.17 mm to (178.2, 106.2)
- moved TP3 0.17 mm to (198.2, 106.2)
Routing:
- net /ZeDMD/BTN_UP: track 0.00 -> 117.9 mm, vias 0 -> 2
- net /ZeDMD/BTN_LEFT: track 0.00 -> 79.4 mm, vias 0 -> 2
- net /LRC: track 0.00 -> 78.3 mm, vias 0 -> 4
- net /ZeDMD/BTN_RIGHT: track 0.00 -> 74.4 mm, vias 0 -> 2
- net /ZeDMD/BTN_DOWN: track 0.00 -> 64.2 mm, vias 0 -> 2
- net /ZeDMD/HUB_OE: track 0.00 -> 57.6 mm, vias 0 -> 1
- net /BCLK: track 0.00 -> 53.2 mm, vias 0 -> 2
- net /MISO: track 0.00 -> 52.9 mm, vias 0 -> 2
- net /MOSI: track 0.00 -> 51.0 mm, vias 0 -> 2
- net /SCK: track 0.00 -> 47.4 mm, vias 0 -> 2
- net /CS: track 0.00 -> 46.2 mm, vias 0 -> 3
- net /ZeDMD/HUB_E: track 0.00 -> 44.6 mm, vias 0 -> 2
- net /ZeDMD/HUB_CLK: track 0.00 -> 42.8 mm, vias 0 -> 2
- net /ZeDMD/HUB_LAT: track 0.00 -> 42.1 mm, vias 0 -> 2
- net /ZeDMD/HUB_D: track 0.00 -> 39.9 mm, vias 0 -> 2
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
Commit message: PCB updates and production files
Routing:
- net GND: vias 0 -> 1
- added copper zone on B.Cu, net GND
- added copper zone on F.Cu, net GND
Other:
- board text added: "0: UP"
- board text added: "1 E"
- board text added: "10: CS"
- board text added: "11: MOSI"
- board text added: "12: SCK"
- board text added: "13: MISO"
- board text added: "14: LRC"
- board text added: "15 G2"
- board text added: "21: DIN"
- board text added: "40 LAT"
- board text added: "42 D"
- board text added: "45: DOWN"
- board text added: "47: RIGHT"
- board text added: "48: LEFT"
- board text added: "5 G1"
- board text added: "8 B"
- board text added: "9:BCLK"
- board text added: "A 18"
- board text added: "B1 6"
- board text added: "B2 16"
- board text added: "C 3"
- board text added: "CLK 41"
- board text added: "OE 2"
- board text added: "R1 4"
- board text added: "R2 7"
- board text added: "SD"
- board text added: "VBUS 5V"
- board text added: "VCC"
- board text added: "Vin"
- board text removed: "1"
