File: KiCad/ZeDMD_WiFi/ESP32-S3-N16R8.kicad_sch (KiCad schematic)
At the start: 2 parts, among them U1 ESP32-S3-DevKitC

Commit message: Update PCB to Rev1.3
Connections:
- net GPIO17: now reaches U1.10 (GPIO17/ADC2_CH6)
- net GPIO38: now reaches U1.35 (GPIO38)
- net GPIO39: now reaches U1.36 (GPIO39/MTCK)
- no-connect marks 0 -> 3
Other:
- note added: "Do not use GPIO 33-37! In use by internal Flash and PSRAM"
Changed lines of the file:
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@@
 	(title_block
 		(title "YD-ESP32-S3 N16R8")
-		(date "2026-07-11")
-		(rev "1.2")
+		(date "2026-09-04")
+		(rev "1.3")
 		(company "elabree")
-		(comment 1 "https://github.com/jens-b/ZeDMD-5.1.8-WIFI-128x32")
+		(comment 1 "https://github.com/jens-b/The-Arcade")
 		(comment 2 "https://ppuc.github.io/docs/zedmd/")
 		(comment 3 "https://github.com/PPUC/ZeDMD")
+	)
+	(text "Do not use GPIO 33-37!\nIn use by internal Flash and PSRAM"
+		(exclude_from_sim no)
+		(at 186.182 120.396 0)
+		(effects
+			(font
+				(size 1.27 1.27)
+			)
+		)
 	)
 	(junction
@@
 		(color 0 0 0 0)
 	)
+	(no_connect
+		(at 165.1 123.19)
+	)
+	(no_connect
+		(at 165.1 120.65)
+	)
+	(no_connect
+		(at 165.1 118.11)
+	)
 	(wire
 		(pts
@@
 	(wire
 		(pts
+			(xy 160.02 123.19) (xy 165.1 123.19)
+		)
+		(stroke
+			(width 0)
+			(type default)
+		)
+	)
+	(wire
+		(pts
 			(xy 160.02 133.35) (xy 177.8 133.35)
 		)
@@
 	(wire
 		(pts
+			(xy 160.02 125.73) (xy 177.8 125.73)
+		)
+		(stroke
+			(width 0)
+			(type default)
+		)
+	)
+	(wire
+		(pts
 			(xy 118.11 38.1) (xy 133.35 38.1)
 		)
@@
 	(wire
 		(pts
+			(xy 160.02 118.11) (xy 165.1 118.11)
+		)
+		(stroke
+			(width 0)
+			(type default)
+		)
+	)
+	(wire
+		(pts
 			(xy 88.9 77.47) (xy 109.22 77.47)
 		)
@@
 	(wire
 		(pts
+			(xy 160.02 110.49) (xy 177.8 110.49)
+		)
+		(stroke
+			(width 0)
+			(type default)
+		)
+	)
+	(wire
+		(pts
 			(xy 127 146.05) (xy 134.62 146.05)
 		)
@@
 	(wire
 		(pts
+			(xy 160.02 120.65) (xy 165.1 120.65)
+		)
+		(stroke
+			(width 0)
+			(type default)
+		)
+	)
+	(wire
+		(pts
 			(xy 163.83 46.99) (xy 163.83 72.39)
 		)
@@
 		(pts
 			(xy 160.02 72.39) (xy 163.83 72.39)
+		)
+		(stroke
+			(width 0)
+			(type default)
+		)
+	)
+	(wire
+		(pts
+			(xy 88.9 72.39) (xy 109.22 72.39)
 		)
 		(stroke
@@
 		)
 	)
+	(hierarchical_label "GPIO39"
+		(shape bidirectional)
+		(at 88.9 72.39 180)
+		(effects
+			(font
+				(size 1.27 1.27)
+			)
+			(justify right)
+		)
+	)
+	(hierarchical_label "GPIO38"
+		(shape bidirectional)
+		(at 177.8 125.73 0)
+		(effects
+			(font
+				(size 1.27 1.27)
+			)
+			(justify left)
+		)
+	)
 	(hierarchical_label "GPIO16"
 		(shape output)
@@
 		(effects
 			(font
+				(size 1.27 1.27)
+			)
+			(justify left)
+		)
+	)
+	(hierarchical_label "GPIO17"
+		(shape input)
+		(at 177.8 110.49 0)
+		(effects
+			(font
